File: hardware/hardware.kicad_pcb (KiCad board)
At the start: 2 copper layers, 100 x 100 mm, 166 parts, among them J1 Conn_01x04_Pin, J10 Conn_01x03, J11 Conn_02x03_Odd_Even, J12 Conn_01x03, J13 Conn_01x03, J14 Conn_01x03, J15 Conn_02x05_Odd_Even, J16 Conn_01x02, J17 RJ45_Hanrun_HR911105A_Horizon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, J18 Conn_01x04, J19 Conn_02x05_Odd_Even, J2 Conn_01x04_Pin, J3 Conn_01x04_Pin, J4 Conn_01x04_Pin, J5 Conn_01x04_Pin, J6 Conn_01x04_Pin, J7 Conn_01x04_Pin, J8 Conn_01x03, J9 Conn_01x02, K1 G5Q-1, K3 G5Q-1, P1 USB_C_Plug, Q1 AO3400A, Q2 AO3400A, U1 DRV8825PWPR, U10 TPS562200, U11 LM317_SOT-223, U2 DRV8825PWPR, U3 DRV8825PWPR, U4 DRV8825PWPR, U5 DRV8825PWPR, U6 DRV8825PWPR, U7 DRV8825PWPR, Y1 Crystal_GND24

Commit message: vbus to 3.3 on DRV
Parts:
- added C31: 47uF, Capacitor_SMD:CP_Elec_6.3x9.9, F.Cu at (64.6, 82.2)
- added C32: 3.3uf, Capacitor_SMD:C_0603_1608Metric, F.Cu at (71.8, 79.6)
- added C33: 3.3uf, Capacitor_SMD:C_0603_1608Metric, F.Cu at (77.2, 87.4)
- added C34: 0.1uF, Capacitor_SMD:C_0603_1608Metric, F.Cu at (77.2, 89.0)
- added C35: 3.3uf, Capacitor_SMD:C_0603_1608Metric, F.Cu at (77.2, 90.6)
- added U13: SSP1117-3.3V, Package_TO_SOT_SMD:SOT-223-3_TabPin2, F.Cu at (76.4, 82.0)
- moved C67 53.2 mm to (88.7, 98.8), turned to -90 degrees
- moved C55 51.0 mm to (87.0, 98.8), turned to -90 degrees
- moved C68 50.2 mm to (87.1, 115.8), turned to 180 degrees
- moved C69 40.5 mm to (73.0, 97.6)
- moved C30 39.8 mm to (75.4, 95.5), turned to 90 degrees
- moved BZ1 22.3 mm to (56.4, 130.0), turned to -90 degrees
Connections:
- JP1 pad 3: +5V -> +3V3
- JP10 pad 3: +5V -> +3V3
- JP11 pad 3: +5V -> +3V3
- JP12 pad 3: +5V -> +3V3
- JP13 pad 3: +5V -> +3V3
- JP14 pad 3: +5V -> +3V3
- JP15 pad 3: +5V -> +3V3
- JP16 pad 3: +5V -> +3V3
- JP17 pad 3: +5V -> +3V3
- JP18 pad 3: +5V -> +3V3
- JP19 pad 3: +5V -> +3V3
- JP2 pad 3: +5V -> +3V3
- JP20 pad 3: +5V -> +3V3
- JP21 pad 3: +5V -> +3V3
- JP3 pad 3: +5V -> +3V3
- JP4 pad 3: +5V -> +3V3
- JP5 pad 3: +5V -> +3V3
- JP6 pad 3: +5V -> +3V3
- JP7 pad 3: +5V -> +3V3
- JP8 pad 3: +5V -> +3V3
- JP9 pad 3: +5V -> +3V3
- RV1 pad 1: 3.3_1 -> +3V3
- RV2 pad 1: 3.3_2 -> +3V3
- RV3 pad 1: 3.3_3 -> +3V3
- RV4 pad 1: 3.3_4 -> +3V3
- RV5 pad 1: 3.3_5 -> +3V3
- RV6 pad 1: 3.3_6 -> +3V3
- RV7 pad 1: 3.3_7 -> +3V3
- U8 pad 29: SPI1_NSS -> unconnected-(U8-PA4/ADC4/DAC0-Pad29)
- U8 pad 30: SPI1_SCK -> unconnected-(U8-PA5/ADC5/DAC1-Pad30)
- U8 pad 31: SPI1_MISO -> unconnected-(U8-PA6/ADC6-Pad31)
- U8 pad 32: SPI1_MOSI -> unconnected-(U8-PA7/ADC7-Pad32)
Routing:
- net +5V: track 424.4 -> 304.5 mm
- net DIR_2: track 26.3 -> 88.0 mm, vias 1 -> 4
- net DIR_4: track 18.7 -> 70.8 mm, vias 1 -> 6
- net SERVO_3: track 0.00 -> 49.3 mm, vias 0 -> 1
- net +3V3: track 22.4 -> 65.1 mm, vias 0 -> 7
- net STEP_2: track 27.3 -> 64.1 mm, vias 1 -> 4
- net BOOT1: track 0.00 -> 31.4 mm, vias 0 -> 1
- net Net-(J17-Pad12): track 35.3 -> 9.15 mm, vias 1 -> 0
- net LED_BLUE: track 8.91 -> 1.53 mm, vias 2 -> 1
- net LED_RED: track 9.39 -> 2.33 mm, vias 2 -> 1
- net GND: track 40.7 -> 47.0 mm
- net BOOT0: track 0.00 -> 6.04 mm
- net unconnected-(J17-NC-Pad7): track 5.86 -> 0.00 mm
- net XTAL1: track 5.95 -> 8.49 mm
- net XTAL2: track 6.02 -> 8.54 mm
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- added copper zone on In2.Cu, net +3V3
- added copper zone on In1.Cu, net GND
Other:
- copper layers 2 -> 4

Commit message: finish PCB
Parts:
- moved C70 0.80 mm to (69.8, 114.6), turned to 180 degrees
- moved C74 0.63 mm to (69.4, 117.0)
- moved C75 0.62 mm to (71.2, 117.0)
- moved RST1 0.15 mm to (70.8, 121.4)
Connections:
- R11 pad 2: +5V -> +3V3
- R12 pad 2: +5V -> +3V3
- R19 pad 2: +5V -> +3V3
- R20 pad 2: +5V -> +3V3
- R21 pad 2: +5V -> +3V3
- R22 pad 2: +5V -> +3V3
- R23 pad 2: +5V -> +3V3
- R24 pad 2: +5V -> +3V3
- R27 pad 2: +5V -> +3V3
- R28 pad 2: +5V -> +3V3
- R4 pad 2: +5V -> +3V3
- R8 pad 2: +5V -> +3V3
- U1 pad 16: +5V -> +3V3
- U1 pad 17: +5V -> +3V3
- U2 pad 16: +5V -> +3V3
- U2 pad 17: +5V -> +3V3
- U3 pad 16: +5V -> +3V3
- U3 pad 17: +5V -> +3V3
- U4 pad 16: +5V -> +3V3
- U4 pad 17: +5V -> +3V3
- U5 pad 16: +5V -> +3V3
- U5 pad 17: +5V -> +3V3
- U6 pad 16: +5V -> +3V3
- U6 pad 17: +5V -> +3V3
- U7 pad 16: +5V -> +3V3
- U7 pad 17: +5V -> +3V3
- U8 pad 4: unconnected-(U8-PE5-Pad4) -> RELAY_1
- U8 pad 5: unconnected-(U8-PE6-Pad5) -> RELAY_2
Routing:
- net +3V3: track 65.1 -> 298.8 mm, vias 7 -> 29
- net +5V: track 304.5 -> 74.2 mm
- net RELAY_1: track 3.18 -> 30.0 mm
- net LED_BLUE: track 1.53 -> 28.2 mm, vias 1 -> 2
- net LED_RED: track 2.33 -> 27.0 mm, vias 1 -> 2
- net 3.3_5: track 21.9 -> 2.33 mm
- net 3.3_7: track 21.2 -> 2.20 mm
- net 3.3_4: track 21.0 -> 2.13 mm
- net 3.3_6: track 20.8 -> 2.11 mm
- net 3.3_1: track 21.0 -> 2.49 mm
- net 3.3_2: track 20.9 -> 2.38 mm
- net 3.3_3: track 20.5 -> 2.16 mm
- net I2C1_SDA: track 0.00 -> 13.2 mm
- net RELAY_2: track 2.47 -> 15.5 mm
- net BOOT0: track 6.04 -> 16.3 mm, vias 0 -> 1
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