File: hardware/hardware.kicad_sch (KiCad schematic)
At the start: 161 parts, among them J1 Conn_01x04_Pin, J10 Conn_01x03, J11 Conn_02x03_Odd_Even, J12 Conn_01x03, J13 Conn_01x03, J14 Conn_01x03, J15 Conn_02x05_Odd_Even, J16 Conn_01x02, J17 RJ45_Hanrun_HR911105A_Horizon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, J18 Conn_01x04, J19 Conn_02x05_Odd_Even, J2 Conn_01x04_Pin, J3 Conn_01x04_Pin, J4 Conn_01x04_Pin, J5 Conn_01x04_Pin, J6 Conn_01x04_Pin, J7 Conn_01x04_Pin, J8 Conn_01x03, J9 Conn_01x02, K1 G5Q-1, K3 G5Q-1, P1 USB_C_Plug, Q1 AO3400A, Q2 AO3400A, U1 DRV8825PWPR, U10 TPS562200, U11 LM317_SOT-223, U2 DRV8825PWPR, U3 DRV8825PWPR, U4 DRV8825PWPR, U5 DRV8825PWPR, U6 DRV8825PWPR, U7 DRV8825PWPR, Y1 Crystal_GND24

Commit message: vbus to 3.3 on DRV
Parts:
- added C31: 47uF, Capacitor_SMD:CP_Elec_6.3x9.9, symbol Device:C_Polarized_US
- added C32, C33, C35: 3.3uf, Capacitor_SMD:C_0603_1608Metric, symbol Device:C_Small
- added C34: 0.1uF, Capacitor_SMD:C_0603_1608Metric, symbol Device:C_Small
- added U13: SSP1117-3.3V, Package_TO_SOT_SMD:SOT-223-3_TabPin2, symbol Regulator_Linear:LM1117MP-3.3
Connections:
- net +3V3: now also JP1.3 (B), JP10.3 (B), JP11.3 (B), JP12.3 (B), JP13.3 (B), JP14.3 (B), JP15.3 (B), JP16.3 (B), JP17.3 (B), JP18.3 (B), JP19.3 (B), JP2.3 (B), JP20.3 (B), JP21.3 (B), JP3.3 (B), JP4.3 (B), JP5.3 (B), JP6.3 (B), JP7.3 (B), JP8.3 (B), JP9.3 (B), RV1.1, RV2.1, RV3.1, RV4.1, RV5.1, RV6.1, RV7.1, C33.2, C34.2, C35.2, U13.2 (VO)
- net +5V: now also C31.1, C32.2, U13.3 (VI); no longer JP1.3 (B), JP10.3 (B), JP11.3 (B), JP12.3 (B), JP13.3 (B), JP14.3 (B), JP15.3 (B), JP16.3 (B), JP17.3 (B), JP18.3 (B), JP19.3 (B), JP2.3 (B), JP20.3 (B), JP21.3 (B), JP3.3 (B), JP4.3 (B), JP5.3 (B), JP6.3 (B), JP7.3 (B), JP8.3 (B), JP9.3 (B)
- net 3.3_1: no longer RV1.1
- net 3.3_2: no longer RV2.1
- net 3.3_3: no longer RV3.1
- net 3.3_4: no longer RV4.1
- net 3.3_5: no longer RV5.1
- net 3.3_6: no longer RV6.1
- net 3.3_7: no longer RV7.1
- net GND: now also C31.2, C32.1, C33.1, C34.1, C35.1, U13.1 (GND)
- net SPI1_MISO: no longer names the net of U8.31 (PA6/ADC6)
- net SPI1_MOSI: no longer names the net of U8.32 (PA7/ADC7)
- net SPI1_NSS: no longer names the net of U8.29 (PA4/ADC4/DAC0)
- net SPI1_SCK: no longer names the net of U8.30 (PA5/ADC5/DAC1)
Other:
- note added: "VOLTAGE REGULATOR / DECOUPLING CAPACITORS"

Commit message: finish PCB
Connections:
- net +3V3: now also R11.2, R12.2, R19.2, R20.2, R21.2, R22.2, R23.2, R24.2, R27.2, R28.2, R4.2, R8.2, U1.16 (~{NRESET}), U1.17 (NSLEEP), U2.16 (~{NRESET}), U2.17 (NSLEEP), U3.16 (~{NRESET}), U3.17 (NSLEEP), U4.16 (~{NRESET}), U4.17 (NSLEEP), U5.16 (~{NRESET}), U5.17 (NSLEEP), U6.16 (~{NRESET}), U6.17 (NSLEEP), U7.16 (~{NRESET}), U7.17 (NSLEEP)
- net +5V: no longer R11.2, R12.2, R19.2, R20.2, R21.2, R22.2, R23.2, R24.2, R27.2, R28.2, R4.2, R8.2, U1.16 (~{NRESET}), U1.17 (NSLEEP), U2.16 (~{NRESET}), U2.17 (NSLEEP), U3.16 (~{NRESET}), U3.17 (NSLEEP), U4.16 (~{NRESET}), U4.17 (NSLEEP), U5.16 (~{NRESET}), U5.17 (NSLEEP), U6.16 (~{NRESET}), U6.17 (NSLEEP), U7.16 (~{NRESET}), U7.17 (NSLEEP)
- net RELAY_1: now also U8.4 (PE5)
- net RELAY_2: now also U8.5 (PE6)
